File: PCB/PCB.kicad_sch (KiCad schematic)
At the start: 28 parts, among them J1 SPI, J10 ESC5, J11 ESC6, J12 ESC7, J13 ESC8, J14 ESC9, J15 ESC10, J16 ESC11, J17 ESC12, J18 Barrel_Jack_Switch, J19 HX711_1, J20 HX711_2, J3 3.3V, J4 GND, J5 PINS, J6 ESC1, J7 ESC2, J8 ESC3, J9 ESC4, U1 pi pico, U2 L7805

Commit message: add PCB layout design
Parts:
- added P1, P10, P11, P12, P2, P3, P4, P5, P6, P7, P8, P9: P1, TerminalBlock:TerminalBlock_bornier-2_P5.08mm, symbol Connector:Screw_Terminal_01x02
- added P_IN1, P_IN2, P_IN3: P, TerminalBlock:TerminalBlock_bornier-2_P5.08mm, symbol Connector:Screw_Terminal_01x02
- 3V3: renamed from J3; footprint (none) -> Connector_PinSocket_2.54mm:PinSocket_1x04_P2.54mm_Vertical
- E1: renamed from J6; footprint (none) -> Connector_PinSocket_2.54mm:PinSocket_1x03_P2.54mm_Vertical
- E10: renamed from J15; footprint (none) -> Connector_PinSocket_2.54mm:PinSocket_1x03_P2.54mm_Vertical
- E11: renamed from J16; footprint (none) -> Connector_PinSocket_2.54mm:PinSocket_1x03_P2.54mm_Vertical
- E12: renamed from J17; footprint (none) -> Connector_PinSocket_2.54mm:PinSocket_1x03_P2.54mm_Vertical
- E2: renamed from J7; footprint (none) -> Connector_PinSocket_2.54mm:PinSocket_1x03_P2.54mm_Vertical
- E3: renamed from J8; footprint (none) -> Connector_PinSocket_2.54mm:PinSocket_1x03_P2.54mm_Vertical
- E4: renamed from J9; footprint (none) -> Connector_PinSocket_2.54mm:PinSocket_1x03_P2.54mm_Vertical
- E5: renamed from J10; footprint (none) -> Connector_PinSocket_2.54mm:PinSocket_1x03_P2.54mm_Vertical
- E6: renamed from J11; footprint (none) -> Connector_PinSocket_2.54mm:PinSocket_1x03_P2.54mm_Vertical
- E7: renamed from J12; footprint (none) -> Connector_PinSocket_2.54mm:PinSocket_1x03_P2.54mm_Vertical
- E8: renamed from J13; footprint (none) -> Connector_PinSocket_2.54mm:PinSocket_1x03_P2.54mm_Vertical
- E9: renamed from J14; footprint (none) -> Connector_PinSocket_2.54mm:PinSocket_1x03_P2.54mm_Vertical
- GND1: renamed from J4; footprint (none) -> Connector_PinSocket_2.54mm:PinSocket_1x04_P2.54mm_Vertical
- J1: footprint Connector_PinSocket_2.54mm:PinSocket_1x04_P2.54mm_Vertical -> Connector_PinSocket_2.54mm:PinSocket_1x06_P2.54mm_Vertical
- LC1: renamed from J19; footprint (none) -> Connector_PinSocket_2.54mm:PinSocket_1x04_P2.54mm_Vertical
- LC2: renamed from J20; footprint (none) -> Connector_PinSocket_2.54mm:PinSocket_1x04_P2.54mm_Vertical
- PINS1: renamed from J5; footprint (none) -> Connector_PinSocket_2.54mm:PinSocket_1x04_P2.54mm_Vertical
- U1: footprint RaspberryPi:raspberry pi pico -> pipico:raspberry pi pico
Connections:
- net GND: now also P1.2 (Pin_2), P10.2 (Pin_2), P11.2 (Pin_2), P12.2 (Pin_2), P2.2 (Pin_2), P3.2 (Pin_2), P4.2 (Pin_2), P5.2 (Pin_2), P6.2 (Pin_2), P7.2 (Pin_2), P8.2 (Pin_2), P9.2 (Pin_2), P_IN1.2 (Pin_2), P_IN2.2 (Pin_2), P_IN3.2 (Pin_2)
- new net: P1.1 (Pin_1), P2.1 (Pin_1), P3.1 (Pin_1), P4.1 (Pin_1), P_IN1.1 (Pin_1)
- new net: P5.1 (Pin_1), P6.1 (Pin_1), P7.1 (Pin_1), P8.1 (Pin_1), P_IN2.1 (Pin_1)
- new net: P10.1 (Pin_1), P11.1 (Pin_1), P12.1 (Pin_1), P9.1 (Pin_1), P_IN3.1 (Pin_1)
Other:
- note added: "ESC POWER"
- moved on the sheet: 3V3, GND1, J1, PINS1
