File: PCB/PCB.kicad_pcb (KiCad board)
At the start: 2 copper layers, 99.1 x 99.1 mm, 45 parts, among them J1 SPI, J18 Barrel_Jack_Switch, P1 P1, P10 P1, P11 P1, P12 P1, P2 P1, P3 P1, P4 P1, P5 P1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

Commit message: fix and add production files
Parts:
- moved 3V3 2.22 mm to (122.6, 90.2)
- moved GND1 1.42 mm to (126.4, 90.2)
- moved PINS1 0.64 mm to (130.2, 90.2)
Routing:
- net GND: track 0.00 -> 5.07 mm, vias 0 -> 28
- net PIN15: track 7.87 -> 7.24 mm
- net PIN14: track 7.87 -> 7.24 mm
- net PIN13: track 8.92 -> 8.29 mm
- net PIN12: track 8.92 -> 8.29 mm
- added copper zone on B.Cu, net +3V3
- added copper zone on F.Cu, net Net-(P1-Pin_1)
- added copper zone on F.Cu, net Net-(P10-Pin_1)
- added copper zone on F.Cu, net Net-(P5-Pin_1)
Other:
- board text added: "+ -"
- board text added: "P12"
- board text added: "P13"
- board text added: "P14"
- board text added: "P15"
- board text added: "PINS"
- board text added: "SIG"
- board text added: "VCC"
